File: hzbugger.kicad_sch (KiCad schematic)
At the start: 23 parts, among them J1 USB_A, J2 IDC, U1 STM32F103C8Tx, U2 SRV05-4, U3 AMS1117-3.3, Y1 8M

Commit message: routing
Parts:
- added C11, C12: 22p, Capacitor_SMD:C_0603_1608Metric, symbol Device:C_Small
- added C13: 100n, symbol Device:C_Small
- added C14, C15, C16: 100n, Capacitor_SMD:C_0805_2012Metric, symbol Device:C_Small
- added D1: PWR_LED, LED_SMD:LED_0603_1608Metric, symbol Device:LED
- added D3: LED1, LED_SMD:LED_0603_1608Metric, symbol Device:LED
- added D4: LED2, LED_SMD:LED_0603_1608Metric, symbol Device:LED
- added H1, H2: H1, MountingHole:MountingHole_3.2mm_M3_DIN965_Pad_TopBottom, symbol Mechanical:MountingHole_Pad
- added J3: BOOT0-HDR, Connector_PinHeader_2.54mm:PinHeader_1x03_P2.54mm_Vertical, symbol Connector:Conn_01x03_Pin
- added J4: SWD, Connector_PinHeader_2.54mm:PinHeader_1x04_P2.54mm_Vertical, symbol Connector:Conn_01x04_Pin
- added J5: DC, Connector_PinHeader_2.54mm:PinHeader_1x02_P2.54mm_Vertical, symbol Connector:Conn_01x02_Pin
- added J6: SPI, Connector_PinHeader_2.54mm:PinHeader_1x04_P2.54mm_Vertical, symbol Connector:Conn_01x04_Pin
- added R10, R9: 22R, Resistor_SMD:R_0603_1608Metric, symbol Device:R_Small
- added R11, R7, R8: 10k, Resistor_SMD:R_0805_2012Metric, symbol Device:R_Small
- added R12: 10k, Resistor_SMD:R_0603_1608Metric, symbol Device:R_Small
- added R13: 1k, Resistor_SMD:R_0603_1608Metric, symbol Device:R_Small
- added R6: 4k7, Resistor_SMD:R_0805_2012Metric, symbol Device:R_Small
- C10, C2, C7, C9: footprint (none) -> Capacitor_SMD:C_0805_2012Metric
- C5: footprint (none) -> Resistor_SMD:R_0805_2012Metric
- C6: footprint (none) -> Resistor_SMD:R_0805_2012Metric_Pad1.20x1.40mm_HandSolder
- C8: footprint (none) -> Capacitor_Tantalum_SMD:CP_EIA-6032-15_Kemet-U_Pad2.25x2.35mm_HandSolder
- D2: footprint (none) -> Diode_SMD:D_SMA
- F1: footprint (none) -> Fuse:Fuse_1206_3216Metric_Pad1.42x1.75mm_HandSolder; LCSC (none) -> DNP
- R2, R3, R4, R5: footprint Resistor_SMD:R_0805_2012Metric -> Resistor_SMD:R_0603_1608Metric
- U1: value STM32F103C8Tx -> STM32F103C8T6; LCSC (none) -> C8734
Connections:
- net +3V3: now also C2.1, J2.8 (Pin_8), C13.1, C15.1, C16.1, D4.2 (A), J3.1 (Pin_1), J4.2 (Pin_2), J5.2 (Pin_2), R11.2
- net +5V: now also J2.9 (Pin_9), C14.1, R6.1
- net GND: now also C2.2, J2.10 (Pin_10), J2.5 (Pin_5), C11.1, C12.1, C13.2, C14.2, C15.2, C16.2, D1.1 (K), D3.1 (K), H1.1, H2.1, J3.3 (Pin_3), J4.1 (Pin_1), J5.1 (Pin_1), R12.1
- net USB_DM: now also U1.32 (PA11)
- net USB_DP: now also U1.33 (PA12), R11.1
- net LED_LINK: now reaches R3.1
- net LED_LINK: now also U1.30 (PA9), R13.1
- net at R3.2: now also D4.1 (K)
- net at Y1.1: now also U1.6 (PD1), C11.2
- net at Y1.2: now also U1.5 (PD0), C12.2
- net UART_TX: now reaches J2.1 (Pin_1)
- net UART_TX: now also R9.2
- net UART_RX: now reaches J2.2 (Pin_2)
- net UART_RX: now also R10.2
- net SWO_TRACE: now reaches J2.3 (Pin_3)
- net SWO_TRACE: now also U1.43 (PB7)
- net RST: now reaches J2.4 (Pin_4)
- net RST: now also U1.18 (PB0)
- net SWDIO: now reaches J2.6 (Pin_6)
- net SWDIO: now also U1.27 (PB14)
- net SWCLK: now reaches J2.7 (Pin_7)
- net SWCLK: now also U1.15 (PA5)
- net at U1.12 (PA2): now also R9.1
- net at U1.13 (PA3): now also R10.1
- net at U1.20 (PB2): now also R12.2
- net DIO: now reaches U1.34 (PA13)
- net DIO: now also J4.4 (Pin_4)
- net DCLK: now reaches U1.37 (PA14)
- net DCLK: now also J4.3 (Pin_3)
- net at U1.44 (BOOT0): now also R8.1
- new net: D3.2 (A), R13.2
- new net: J3.2 (Pin_2), R8.2
- new net: D1.2 (A), R6.2
Other:
- moved on the sheet: J2, R3, Y1

Commit message: save
Parts:
- added H3: MountingHole, MountingHole:MountingHole_5.3mm_M5_ISO7380, symbol Mechanical:MountingHole
- added J7: SWDOUT_HDR, Connector_PinHeader_2.54mm:PinHeader_1x05_P2.54mm_Horizontal, symbol Connector:Conn_01x05_Pin
Connections:
- net +3V3: now also J7.5 (Pin_5)
- net GND: now also J7.1 (Pin_1)
- net RST: now also J7.2 (Pin_2)
- net SWCLK: now also J7.4 (Pin_4)
- net SWDIO: now also J7.3 (Pin_3)

Commit message: routing
Parts:
- H3: footprint MountingHole:MountingHole_5.3mm_M5_ISO7380 -> MountingHole:MountingHole_5.3mm_M5_Pad
Other:
- note added: "RESET-NAPPI!"
Changed lines of the file:
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@@
+		)
+	)
+	(text "RESET-NAPPI!"
+		(exclude_from_sim no)
+		(at 135.89 149.606 0)
+		(effects
+			(font
+				(size 5 5)
+				(thickness 1)
+				(bold yes)
+			)
 		)
 	)
@@
 			)
 		)
-		(property "Footprint" "MountingHole:MountingHole_5.3mm_M5_ISO7380"
+		(property "Footprint" "MountingHole:MountingHole_5.3mm_M5_Pad"
 			(at 161.29 161.29 0)
 			(effects

Commit message: save
Parts:
- C4: footprint (none) -> Capacitor_SMD:C_0805_2012Metric
- C6: footprint Resistor_SMD:R_0805_2012Metric_Pad1.20x1.40mm_HandSolder -> Capacitor_SMD:C_0805_2012Metric
Changed lines of the file:
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@@
 			)
 		)
-		(property "Footprint" ""
+		(property "Footprint" "Capacitor_SMD:C_0805_2012Metric"
 			(at 83.82 35.56 0)
 			(effects
@@
 			)
 		)
-		(property "Footprint" "Resistor_SMD:R_0805_2012Metric_Pad1.20x1.40mm_HandSolder"
+		(property "Footprint" "Capacitor_SMD:C_0805_2012Metric"
 			(at 205.74 33.02 0)
 			(effects

Commit message: silks etc
Parts:
- added TP1: 5Vtp, TestPoint:TestPoint_Pad_D2.0mm, symbol Connector:TestPoint
- added TP2: 3V3tp, TestPoint:TestPoint_Pad_D2.0mm, symbol Connector:TestPoint
- H3: footprint MountingHole:MountingHole_5.3mm_M5_Pad -> MountingHole:MountingHole_3.2mm_M3_Pad_TopBottom
Connections:
- net +3V3: now also TP2.1
- net +5V: now also TP1.1
Other:
- note added: "GPIO pads"
- note added: "LED silks"
- note added: "SPI/I2C"
Changed lines of the file:
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@@
 	)
 	(junction
+		(at 255.27 30.48)
+		(diameter 0)
+		(color 0 0 0 0)
+	)
+	(junction
 		(at 144.78 48.26)
 		(diameter 0)
@@
 	)
 	(junction
+		(at 121.92 33.02)
+		(diameter 0)
+		(color 0 0 0 0)
+	)
+	(junction
 		(at 269.24 30.48)
 		(diameter 0)
@@
 	(wire
 		(pts
-			(xy 125.73 33.02) (xy 118.11 33.02)
+			(xy 125.73 33.02) (xy 121.92 33.02)
 		)
 		(stroke
@@
 	(wire
 		(pts
-			(xy 259.08 30.48) (xy 247.65 30.48)
+			(xy 259.08 30.48) (xy 255.27 30.48)
 		)
 		(stroke
@@
 	(wire
 		(pts
+			(xy 121.92 33.02) (xy 118.11 33.02)
+		)
+		(stroke
+			(width 0)
+			(type default)
+		)
+	)
+	(wire
+		(pts
 			(xy 166.37 91.44) (xy 160.02 91.44)
 		)
@@
 	(wire
 		(pts
+			(xy 255.27 30.48) (xy 247.65 30.48)
+		)
+		(stroke
+			(width 0)
+			(type default)
+		)
+	)
+	(wire
+		(pts
 			(xy 139.7 34.29) (xy 139.7 35.56)
 		)
@@
 		)
 	)
+	(text "SPI/I2C"
+		(exclude_from_sim no)
+		(at 100.584 164.592 0)
+		(effects
+			(font
+				(size 5 5)
+				(thickness 1)
+				(bold yes)
+			)
+		)
+	)
+	(text "GPIO pads\n"
+		(exclude_from_sim no)
+		(at 55.626 182.118 0)
+		(effects
+			(font
+				(size 5 5)
+				(thickness 1)
+				(bold yes)
+			)
+		)
+	)
 	(text "RESET-NAPPI!"
 		(exclude_from_sim no)
@@
 		)
 	)
+	(text "LED silks"
+		(exclude_from_sim no)
+		(at 60.452 155.702 0)
+		(effects
+			(font
+				(size 5 5)
+				(thickness 1)
+				(bold yes)
+			)
+		)
+	)
 	(global_label "DIO"
 		(shape input)
@@
 			)
 		)
-		(property "Footprint" "MountingHole:MountingHole_5.3mm_M5_Pad"
+		(property "Footprint" "MountingHole:MountingHole_3.2mm_M3_Pad_TopBottom"
 			(at 161.29 161.29 0)
 			(effects
@@
 	)
 	(symbol
+		(lib_id "Connector:TestPoint")
+		(at 255.27 30.48 0)
+		(unit 1)
+		(exclude_from_sim no)
+		(in_bom yes)
+		(on_board yes)
+		(dnp no)
+		(fields_autoplaced yes)
+		(property "Reference" "TP2"
+			(at 257.81 25.9079 0)
+			(effects
+				(font
+					(size 1.27 1.27)
+				)
+				(justify left)
+			)
+		)
+		(property "Value" "3V3tp"
+			(at 257.81 28.4479 0)
+			(effects
+				(font
+					(size 1.27 1.27)
+				)
+				(justify left)
+			)
+		)
+		(property "Footprint" "TestPoint:TestPoint_Pad_D2.0mm"
+			(at 260.35 30.48 0)
+			(effects
+				(font
+					(size 1.27 1.27)
+				)
+				(hide yes)
+			)
+		)
+		(property "Datasheet" "~"
+			(at 260.35 30.48 0)
+			(effects
+				(font
+					(size 1.27 1.27)
+				)
+				(hide yes)
+			)
+		)
+		(property "Description" "test point"
+			(at 255.27 30.48 0)
+			(effects
+				(font
+					(size 1.27 1.27)
+				)
+				(hide yes)
+			)
+		)
+		(pin "1"
+		)
+		(instances
+			(project "hzbugger"
+				(path "/493ccddd-ac13-43bb-97a7-ed9a2ed970cc"
+					(reference "TP2")
+					(unit 1)
+				)
+			)
+		)
+	)
+	(symbol
 		(lib_id "Device:R_Small")
 		(at 105.41 88.9 90)
@@
 					(unit 1)
 				)
+			)
+		)
+	)
+	(symbol
+		(lib_id "Connector:TestPoint")
+		(at 121.92 33.02 0)
+		(unit 1)
+		(exclude_from_sim no)
+		(in_bom yes)
+		(on_board yes)
+		(dnp no)
+		(property "Reference" "TP1"
+			(at 124.46 28.4479 0)
+			(effects
+				(font
+					(size 1.27 1.27)
+				)
+				(justify left)
+			)
+		)
+		(property "Value" "5Vtp"
+			(at 117.602 24.638 0)
+			(effects
+				(font
+					(size 1.27 1.27)
+				)
+				(justify left)
+			)
+		)
+		(property "Footprint" "TestPoint:TestPoint_Pad_D2.0mm"
+			(at 127 33.02 0)
+			(effects
+				(font
+					(size 1.27 1.27)
+				)
+				(hide yes)
+			)
+		)
+		(property "Datasheet" "~"
+			(at 127 33.02 0)
+			(effects
+				(font
+					(size 1.27 1.27)
+				)
+				(hide yes)
+			)
+		)
+		(property "Description" "test point"
+			(at 121.92 33.02 0)
+			(effects
+				(font
+					(size 1.27 1.27)
+				)
+				(hide yes)
+			)
+		)
+		(pin "1"
+		)
+		(instances
+			(project ""
+				(path "/493ccddd-ac13-43bb-97a7-ed9a2ed970cc"
+					(reference "TP1")
+					(unit 1)
+				)

Commit message: right USB connector, etc
Parts:
- removed J1: USB_A, Connector_USB:USB_A_Kycon_KUSBX-AS1N-B_Horizontal, symbol Connector:USB_A
- added C17: 100n, Capacitor_SMD:C_0603_1608Metric, symbol Device:C_Small
- added H4: MountingHole, MountingHole:MountingHole_3.2mm_M3_Pad_TopBottom, symbol Mechanical:MountingHole
- added R14: 22R, Resistor_SMD:R_0603_1608Metric, symbol Device:R_Small
- added TP3: GNDtp1, TestPoint:TestPoint_Loop_D1.80mm_Drill1.0mm_Beaded, symbol Connector:TestPoint
- added TP4: IOPAD1, TestPoint:TestPoint_Pad_D1.0mm, symbol Connector:TestPoint
- added TP5: IOPAD2, TestPoint:TestPoint_Pad_D1.0mm, symbol Connector:TestPoint
- added TP6: GNDpad, TestPoint:TestPoint_Pad_D2.0mm, symbol Connector:TestPoint
- added U4: HX AM 90D, hzbugger:USB-A-TH_HANXIA_HXAM90D, symbol hzbugger:HXAM90D
- C1, C13, C3: footprint (none) -> Capacitor_SMD:C_0603_1608Metric
- C10, C14, C15, C16, C2, C7, C9: footprint Capacitor_SMD:C_0805_2012Metric -> Capacitor_SMD:C_0603_1608Metric
- C5: footprint Resistor_SMD:R_0805_2012Metric -> Capacitor_SMD:C_0603_1608Metric
- D1, D3, D4: footprint LED_SMD:LED_0603_1608Metric -> LED_THT:LED_D3.0mm
- R1: value 10k -> 22R; footprint Resistor_SMD:R_0805_2012Metric -> Resistor_SMD:R_0603_1608Metric
- R11: value 10k -> 1k5; footprint Resistor_SMD:R_0805_2012Metric -> Resistor_SMD:R_0603_1608Metric
- R6: value 4k7 -> 470R
- TP2: value 3V3tp -> NRST
Connections:
- net +3V3: now also U1.1 (VBAT); no longer TP2.1
- net GND: now also J6.1 (Pin_1), C17.1, TP3.1, TP6.1, U4.4 (GND), U4.5 (EH), U4.6 (EH)
- net USB_DP: now also U2.6 (IO4); no longer U2.1 (IO1)
- net VBUS: now also U4.1 (VCC)
- net at R5.1: now also U4.2 (D-)
- net at J6.2 (Pin_2): now also R1.2
- net at J6.3 (Pin_3): now also R2.2
- net at J6.4 (Pin_4): now also R14.2
- net at R7.1: now also TP2.1
- net at R7.2: now also U1.7 (NRST), C17.2
- net at R4.1: now also U4.3 (D+)
- net SPI1_SCK: now reaches R1.1
- net SPI1_SCK: now also U1.39 (PB3)
- net SPI1_MISO: now reaches R2.1
- net SPI1_MISO: now also U1.40 (PB4)
- net SPI1_MOSI: now reaches U1.41 (PB5)
- net SPI1_MOSI: now also R14.1
- net at U1.45 (PB8): now also TP4.1
- net at U1.46 (PB9): now also TP5.1
Other:
- note added: "RESET-NAPPI! BOOT-nappi?"
- note removed: "GPIO pads"
- note removed: "LED silks"
- note removed: "RESET-NAPPI!"
- note removed: "SPI/I2C"
- moved on the sheet: C13, J5, R4, R5, R7

Commit message: LCSC codes
Parts:
- removed TP6: GNDpad, TestPoint:TestPoint_Pad_D2.0mm, symbol Connector:TestPoint
- added R15, R18: 0R, Resistor_SMD:R_0603_1608Metric_Pad0.98x0.95mm_HandSolder, symbol Device:R_Small
- added R16: 0R, Resistor_SMD:R_0603_1608Metric, symbol Device:R_Small
- C1, C10, C13, C14, C15, C16, C17, C2, C3, C5, C7, C9: LCSC (none) -> C14663
- C11, C12: LCSC (none) -> C1653
- C4, C6: LCSC (none) -> C15850
- C8: LCSC (none) -> DNP; now not fitted
- D2: LCSC (none) -> C8678
- F1: now not fitted
- J6: value SPI -> GPIO; footprint Connector_PinHeader_2.54mm:PinHeader_1x04_P2.54mm_Vertical -> Connector_PinHeader_2.54mm:PinHeader_1x06_P2.54mm_Vertical; symbol Connector:Conn_01x04_Pin -> Connector:Conn_01x06_Pin
- R1, R14, R2, R4, R5, R9: LCSC (none) -> C23345
- R10: footprint Resistor_SMD:R_0603_1608Metric -> Resistor_SMD:R_0603_1608Metric_Pad0.98x0.95mm_HandSolder; LCSC (none) -> C23345
- R11: LCSC (none) -> C22843
- R12: LCSC (none) -> C25804
- R13, R3: value 1k -> 470R; LCSC (none) -> C23179
- R6: footprint Resistor_SMD:R_0805_2012Metric -> Resistor_SMD:R_0603_1608Metric_Pad0.98x0.95mm_HandSolder; LCSC (none) -> C23179
- R7, R8: footprint Resistor_SMD:R_0805_2012Metric -> Resistor_SMD:R_0603_1608Metric; LCSC (none) -> C25804
- U2: LCSC (none) -> C7420376
- U3: LCSC (none) -> C6186
- U4: LCSC (none) -> C5160314; LCSC Part C5160314 -> (none)
- Y1: LCSC (none) -> C12674
Connections:
- net +3V3: now also J6.5 (Pin_5)
- net GND: now also J6.6 (Pin_6)
- net RST: now also R18.1; no longer U1.18 (PB0)
- net SWCLK: now also R15.2; no longer U1.15 (PA5)
- net SWDIO: now also R16.1; no longer U1.27 (PB14)
- new net: R18.2, U1.18 (PB0)
- new net: R15.1, U1.15 (PA5)
- new net: R16.2, U1.27 (PB14)
Other:
- note added: "boot1"
- moved on the sheet: C13, J5, R1, R12, R14, R2, R6
